Commit message: Transform frames currently still being tested

File: src/D435i/D435i/urdf/test_frame.urdf.xacro (robot description, xacro)
@@ -1 +1,77 @@
-/home/ors/ros2_ws/src/D435i/D435i/urdf/test_frame.urdf.xacro
+<?xml version="1.0"?>
+<robot name="test_robot" xmlns:xacro="http://www.ros.org/wiki/xacro">
+  <!-- Declare arguments for frame names -->
+  <xacro:arg name="camera_name" default="camera_link"/>
+  <!-- ===================================================
+       Robot Base Link Definition
+       =================================================== -->
+  <link name="base_link">
+    <!-- Visual representation -->
+    <visual>
+      <geometry>
+        <box size="0.4 0.4 0.1"/>
+      </geometry>
+      <origin xyz="0 0 0.05" rpy="0 0 0"/>
+      <material name="blue">
+        <color rgba="0 0 1 1"/>
+      </material>
+    </visual>
+    <!-- Collision properties -->
+    <collision>
+      <geometry>
+        <box size="0.4 0.4 0.1"/>
+      </geometry>
+      <origin xyz="0 0 0.05" rpy="0 0 0"/>
+    </collision>
+    <!-- Inertial properties -->
+    <inertial>
+      <mass value="5.0"/>
+      <origin xyz="0 0 0.05" rpy="0 0 0"/>
+      <inertia
+        ixx="0.02" ixy="0.0" ixz="0.0"
+        iyy="0.02" iyz="0.0"
+        izz="0.02"/>
+    </inertial>
+  </link>
+  <!-- ===================================================
+       Camera Link Definition
+       =================================================== -->
+  <!-- <link name="${camera_frame}"> -->
+  <link name="{$camera_name}">
+    <!-- Visual representation -->
+    <visual>
+      <geometry>
+        <box size="0.1 0.03 0.03"/>
+      </geometry>
+      <origin xyz="0 0 0" rpy="0 0 0"/>
+      <material name="gray">
+        <color rgba="0.5 0.5 0.5 1"/>
+      </material>
+    </visual>
+    <!-- Collision properties -->
+    <collision>
+      <geometry>
+        <box size="0.1 0.03 0.03"/>
+      </geometry>
+      <origin xyz="0 0 0" rpy="0 0 0"/>
+    </collision>
+    <!-- Inertial properties -->
+    <inertial>
+      <mass value="0.1"/>
+      <origin xyz="0 0 0" rpy="0 0 0"/>
+      <inertia
+        ixx="0.0001" ixy="0.0" ixz="0.0"
+        iyy="0.0001" iyz="0.0"
+        izz="0.0001"/>
+    </inertial>
+  </link>
+  <!-- ===================================================
+       Joint Connecting Camera to Robot Base Link
+       =================================================== -->
+  <joint name="camera_mount_joint" type="fixed">
+    <parent link="base_link"/>
+    <!-- <child link="${camera_frame}"/> -->
+    <child link="robot_link"/>
+    <origin xyz="0 0 0.15" rpy="0 0 0"/>
+  </joint>
+</robot>

Commit message: feat: package containing launch file to launch D435i ROS2 Node with configurable camera frame ID
Removed extra code from d435i.launch.py which was used in testing the configurable camera frame ID feature and will not be necessary during simulation or physical testing
The package also contains the D435i URDF files which may or may not be needed during simulation/testing.

File: src/D435i/D435i/urdf/test_frame.urdf.xacro (robot description, xacro)
@@ -1,6 +1,4 @@
 <?xml version="1.0"?>
 <robot name="test_robot" xmlns:xacro="http://www.ros.org/wiki/xacro">
-  <!-- Declare arguments for frame names -->
-  <xacro:arg name="camera_name" default="camera_link"/>
   <!-- ===================================================
        Robot Base Link Definition
@@ -38,5 +36,5 @@
        =================================================== -->
   <!-- <link name="${camera_frame}"> -->
-  <link name="{$camera_name}">
+  <link name="depthcam_link">
     <!-- Visual representation -->
     <visual>
@@ -72,6 +70,6 @@
     <parent link="base_link"/>
     <!-- <child link="${camera_frame}"/> -->
-    <child link="robot_link"/>
-    <origin xyz="0 0 0.15" rpy="0 0 0"/>
+    <child link="depthcam_link"/>
+    <origin xyz="0 0 0.85" rpy="0 0 0"/>
   </joint>
 </robot>
